File: wren-left/wren-left.kicad_pcb (KiCad board)
At the start: 2 copper layers, 230.3 x 117 mm, 95 parts, among them J1 TRRS_Jack, SW0 Reset, U1 Elite-C

Commit message: Cleanup, re-add drill holes
Parts:
- added REF**: MountingHole_2.2mm_M2_Pad, MountingHole:MountingHole_2.2mm_M2_Pad, F.Cu at (226.2, 111.9)
- added REF**: MountingHole_2.2mm_M2_Pad, MountingHole:MountingHole_2.2mm_M2_Pad, F.Cu at (56.4, 84.1)
- added REF**: MountingHole_2.2mm_M2_Pad, MountingHole:MountingHole_2.2mm_M2_Pad, F.Cu at (56.4, 46.0)
- added REF**: MountingHole_2.2mm_M2_Pad, MountingHole:MountingHole_2.2mm_M2_Pad, F.Cu at (135.0, 46.0)
- added REF**: MountingHole_2.2mm_M2_Pad, MountingHole:MountingHole_2.2mm_M2_Pad, F.Cu at (135.0, 84.1)
- added REF**: MountingHole_2.2mm_M2_Pad, MountingHole:MountingHole_2.2mm_M2_Pad, F.Cu at (211.1, 45.2)
- added REF**: MountingHole_2.2mm_M2_Pad, MountingHole:MountingHole_2.2mm_M2_Pad, F.Cu at (211.1, 83.3)
- moved R1 5.05 mm to (243.7, 38.1)
- moved R2 3.40 mm to (243.7, 43.7)
- moved D32 1.12 mm to (210.3, 91.3)
- moved D12 1.12 mm to (210.3, 53.2)
- moved D42 1.11 mm to (246.0, 108.7)
- moved D10 0.84 mm to (55.6, 36.5)
- moved D20 0.84 mm to (55.6, 55.6)
- moved D30 0.84 mm to (55.6, 74.6)
- moved D40 0.84 mm to (55.6, 93.7)
- moved D19 0.83 mm to (74.6, 55.6)
- moved D29 0.83 mm to (74.6, 74.6)
- moved D39 0.83 mm to (74.6, 93.7)
- moved D9 0.83 mm to (74.6, 36.5)
- moved D38 0.82 mm to (93.7, 93.7)
- moved D18 0.82 mm to (93.7, 55.6)
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Connections:
- ENC1 pad A: (no net) -> LEFT
- ENC1 pad B: (no net) -> RIGHT
- U1 pad 28: (no net) -> RIGHT
- U1 pad 29: (no net) -> LEFT
Routing:
- net GND: track 132.3 -> 92.8 mm, vias 7 -> 3
- net RIGHT: track 0.00 -> 30.1 mm
- net Net-(SW0-Pad1): track 6.50 -> 35.5 mm, vias 0 -> 1
- net LEFT: track 0.00 -> 23.3 mm
- net COL0: track 107.3 -> 118.0 mm, vias 1 -> 2
- net ROW2: track 227.3 -> 219.2 mm
- net ROW3: track 244.4 -> 236.9 mm, vias 1 -> 0
- net ROW0: track 210.7 -> 203.9 mm, vias 1 -> 0
- net VCC: track 76.3 -> 70.3 mm, vias 3 -> 1
- net COL1: track 148.7 -> 154.3 mm, vias 3 -> 1
- net COL3: track 183.9 -> 180.2 mm, vias 2 -> 1
- net COL7: track 210.4 -> 214.0 mm, vias 2 -> 1
- net ROW4: track 132.9 -> 130.2 mm
- net COL2: track 166.3 -> 165.0 mm, vias 5 -> 1
- net COL5: track 174.7 -> 173.5 mm, vias 2 -> 1
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