File: PCBs/wren-right/wren-right.sch (KiCad schematic (older format))
At the start: 63 parts, among them J1 TRRS_Jack, SW0 Reset, U1 Elite C

Commit message: Reposition Rotary Encoder and Create New Right Board
Parts:
- added D10, D17, D18, D19, D20, D27, D28, D29, D30, D37, D38, D39, D40, D7, D8, D9: D_Small, footprints:D_SOD123_axial, symbol Device:D_Small
- added H1, H2, H3, H4, H5, H6, H7: MountingHole, MountingHole:MountingHole_2.2mm_M2_ISO7380, symbol Mechanical:MountingHole
- added MX10, MX17, MX18, MX19, MX20, MX27, MX28, MX29, MX30, MX37, MX38, MX39, MX40, MX7, MX8, MX9: MX-NoLED, MX_Only:MX-1U, symbol MX_Alps_Hybrid:MX-NoLED
- U1: value Elite C -> Elite-C; symbol keebio:Elite-C -> wren-left-rescue:Elite-C-keebio
Connections:
- net COL0: now also MX41.1 (COL), U1.13 (10/PB6); no longer ENC1.S1, U1.7 (4/PD4)
- net COL1: now also MX42.1 (COL), U1.14 (16/PB2); no longer MX41.1 (COL), U1.8 (5/PC6)
- net COL2: now also MX43.1 (COL), U1.15 (14/PB3); no longer MX42.1 (COL), U1.9 (6/PD7)
- net COL3: now also MX44.1 (COL), U1.16 (15/PB1); no longer MX43.1 (COL), U1.10 (7/PE6)
- net COL4: now also ENC1.S2, U1.17 (A0/PF7); no longer MX44.1 (COL), U1.11 (8/PB4)
- net COL5: now also U1.18 (A1/PF6); no longer U1.12 (9/PB5)
- net ROW0: now also U1.1 (TX0/PD3), D10.1 (K), D7.1 (K), D8.1 (K), D9.1 (K); no longer U1.17 (A0/PF7)
- net ROW1: now also U1.2 (RX1/PD2), D17.1 (K), D18.1 (K), D19.1 (K), D20.1 (K); no longer U1.16 (15/PB1)
- net ROW2: now also U1.7 (4/PD4), D27.1 (K), D28.1 (K), D29.1 (K), D30.1 (K); no longer U1.15 (14/PB3)
- net ROW3: now also U1.8 (5/PC6), D37.1 (K), D38.1 (K), D39.1 (K), D40.1 (K); no longer U1.14 (16/PB2)
- net ROW4: now also U1.12 (9/PB5); no longer U1.13 (10/PB6)
- net COL6: now reaches U1.19 (A2/PF5)
- net COL6: now also MX17.1 (COL), MX27.1 (COL), MX37.1 (COL), MX7.1 (COL)
- net COL7: now reaches U1.20 (A3/PF4)
- net COL7: now also MX18.1 (COL), MX28.1 (COL), MX38.1 (COL), MX8.1 (COL)
- net RIGHT: now reaches U1.28 (F1)
- net RIGHT: now also ENC1.B
- net LEFT: now reaches U1.29 (F0)
- net LEFT: now also ENC1.A
- net at MX41.2 (ROW): now also D41.2 (A); no longer D42.2 (A)
- net at MX42.2 (ROW): now also D42.2 (A); no longer D43.2 (A)
- net at MX43.2 (ROW): now also D43.2 (A); no longer D44.2 (A)
- net at MX44.2 (ROW): now also D44.2 (A); no longer D45.2 (A)
- removed net ENC1-OUT: D41.2 (A), ENC1.S2
- new net: D37.2 (A), MX37.2 (ROW)
- new net: D38.2 (A), MX38.2 (ROW)
- new net: D39.2 (A), MX39.2 (ROW)
- new net: D40.2 (A), MX40.2 (ROW)
- new net: D7.2 (A), MX7.2 (ROW)
- new net: D8.2 (A), MX8.2 (ROW)
- new net: D9.2 (A), MX9.2 (ROW)
- new net: D10.2 (A), MX10.2 (ROW)
- new net: D17.2 (A), MX17.2 (ROW)
- new net: D18.2 (A), MX18.2 (ROW)
- new net: D19.2 (A), MX19.2 (ROW)
- new net: D20.2 (A), MX20.2 (ROW)
- new net: D27.2 (A), MX27.2 (ROW)
- new net: D28.2 (A), MX28.2 (ROW)
- new net: D29.2 (A), MX29.2 (ROW)
- new net: D30.2 (A), MX30.2 (ROW)
- new net COL8: MX19.1 (COL), MX29.1 (COL), MX39.1 (COL), MX9.1 (COL), U1.9 (6/PD7)
- new net COL9: MX10.1 (COL), MX20.1 (COL), MX30.1 (COL), MX40.1 (COL), U1.10 (7/PE6)
- new net ENC1-IN: D45.2 (A), ENC1.S1
- no-connect marks 11 -> 5
Other:
- moved on the sheet: MX41, MX42, MX43, MX44, SW0, U1

Commit message: Various Updates
New plates, updated routing on the right side, assorted other changes.
Parts:
- removed D10, D17, D18, D19, D20, D27, D28, D29, D30, D37, D38, D39, D40, D7, D8, D9: D_Small, footprints:D_SOD123_axial, symbol Device:D_Small
- removed H4, H5: MountingHole, MountingHole:MountingHole_2.2mm_M2_ISO7380, symbol Mechanical:MountingHole
- removed MX10, MX17, MX18, MX19, MX20, MX27, MX28, MX29, MX30, MX37, MX38, MX39, MX40, MX7, MX8, MX9: MX-NoLED, MX_Only:MX-1U, symbol MX_Alps_Hybrid:MX-NoLED
- H1, H2, H3, H6, H7: footprint MountingHole:MountingHole_2.2mm_M2_ISO7380 -> MountingHole:MountingHole_5.5mm
- U1: symbol wren-left-rescue:Elite-C-keebio -> wren-right-rescue:Elite-C-keebio-wren-left-rescue
Connections:
- net labels removed: COL6, COL7, COL8, COL9
- wire segments 145 -> 97
- no-connect marks 5 -> 9
Other:
- moved on the sheet: H6, H7

Commit message: Add increased stagger to right side
Changed lines of the file:
@@
 Text GLabel 1800 1450 0    50   Input ~ 0
 ROW0
-Text GLabel 1800 2250 0    50   Input ~ 0
+Text GLabel 1800 2050 0    50   Input ~ 0
 ROW1
 Text GLabel 1800 2350 0    50   Input ~ 0
@@
 Text GLabel 3950 4250 2    50   BiDi ~ 0
 SDA
-Text GLabel 1600 1650 2    50   Output ~ 0
-GND
-Text GLabel 1600 1750 2    50   Output ~ 0
-GND
 NoConn ~ 3200 1450
 NoConn ~ 2500 2950
@@
 Text GLabel 2250 5800 0    50   Input ~ 0
 RIGHT
-$Comp
-L wren-right-rescue:Elite-C-keebio-wren-left-rescue U1
-U 1 1 6071F7CA
-P 2500 2000
-F 0 "U1" H 2500 2815 50  0000 C CNN
-F 1 "Elite-C" H 2500 2724 50  0000 C CNN
-F 2 "footprints:Elite-C" H 2450 2100 50  0001 C CNN
-F 3 "" H 2450 2100 50  0001 C CNN
-	1    2500 2000
-	1    0    0    -1
-$EndComp
 Text GLabel 3200 1950 2    50   Input ~ 0
 LEFT
@@
 NoConn ~ 2600 2950
 NoConn ~ 2700 2950
-NoConn ~ 1800 2050
+NoConn ~ 1800 1550
 NoConn ~ 1800 2150
-NoConn ~ 1800 1550
+NoConn ~ 1800 2250
+$Comp
+L wren-right-rescue:Elite-C-keebio-wren-left-rescue U1
+U 1 1 6071F7CA
+P 2500 2000
+F 0 "U1" H 2500 2815 50  0000 C CNN
+F 1 "Elite-C" H 2500 2724 50  0000 C CNN
+F 2 "footprints:Elite-C" H 2450 2100 50  0001 C CNN
+F 3 "" H 2450 2100 50  0001 C CNN
+	1    2500 2000
+	1    0    0    -1
+$EndComp
+Text GLabel 1800 1650 0    50   Input ~ 0
+GND
+Text GLabel 1800 1750 0    50   Input ~ 0
+GND
 $EndSCHEMATC
