File: PCBs/wren-numpad/wren-numpad.kicad_pcb (KiCad board)
At the start: 2 copper layers, 227.7 x 112.8 mm, 105 parts, among them J1 TRRS_Jack, SW0 Reset, U1 Elite-C

Commit message: Standardize MCU Pins
Parts:
- removed the G*** at (241.3, 76.4) (x2)
- added G***: LOGO, footprints:wren_logo, B.Cu at (241.3, 76.4)
- added G***: LOGO, footprints:wren_logo, F.Cu at (241.3, 76.4)
Connections:
- U1 pad 10: COL9 -> LEFT
- U1 pad 11: Net-(U1-Pad11) -> RIGHT
- U1 pad 24: Net-(U1-Pad24) -> (no net)
- U1 pad 25: Net-(U1-Pad25) -> (no net)
- U1 pad 26: Net-(U1-Pad26) -> (no net)
- U1 pad 27: Net-(U1-Pad27) -> (no net)
- U1 pad 28: RIGHT -> (no net)
- U1 pad 29: LEFT -> COL9
- U1 pad 3: Net-(U1-Pad3) -> GND
- U1 pad 4: Net-(U1-Pad4) -> GND
Routing:
- net LEFT: track 145.7 -> 164.8 mm
- net RIGHT: track 148.0 -> 166.6 mm
- net COL9: track 286.8 -> 283.2 mm, vias 1 -> 2
