File: PCBs/wren-numpad/wren-numpad.sch (KiCad schematic (older format))
At the start: 102 parts, among them J1 TRRS_Jack, SW0 Reset, U1 Elite-C

Commit message: Standardize MCU Pins
Parts:
- MX1, MX10, MX11, MX12, MX13, MX14, MX15, MX16, MX17, MX18, MX19, MX2, MX20, MX21, MX22, MX23, MX24, MX25, MX26, MX27, MX28, MX29, MX3, MX30, MX31, MX32, MX33, MX34, MX35, MX36, MX37, MX38, MX39, MX4, MX40, MX42, MX43, MX44, MX5, MX6, MX7, MX8, MX9: footprint MX_Only:MX-1U -> footprints:SW_MX_reversible
- MX41: footprint MX_Only:MX-2U-FLIPPED-ReversedStabilizers -> footprints:SW_MX_reversible
- U1: symbol wren-left-rescue:Elite-C-keebio -> wren-numpad-rescue:Elite-C-keebio-wren-left-rescue
Connections:
- net COL9: now also U1.29 (F0); no longer U1.10 (7/PE6)
- net GND: now also U1.3 (GND), U1.4 (GND)
- net LEFT: now also U1.10 (7/PE6); no longer U1.29 (F0)
- net RIGHT: now also U1.11 (8/PB4); no longer U1.28 (F1)
