File: PCBs/wren-nav/wren-nav.kicad_pcb (KiCad board)
At the start: 2 copper layers, 208.7 x 112.8 mm, 93 parts, among them J1 TRRS_Jack, SW0 Reset, U1 Elite-C

Commit message: Standardize MCU Pins
Parts:
- removed the G*** at (241.3, 76.4) (x2)
- added D27: D_Small, footprints:D_SOD123_axial, B.Cu at (112.7, 74.6)
- added D29: D_Small, footprints:D_SOD123_axial, B.Cu at (74.7, 74.6)
- added G***: LOGO, footprints:wren_logo, B.Cu at (241.3, 76.4)
- added G***: LOGO, footprints:wren_logo, F.Cu at (241.3, 76.4)
- added MX27: MX-NoLED, footprints:SW_MX_reversible, F.Cu at (104.0, 74.6)
- added MX29: MX-NoLED, footprints:SW_MX_reversible, F.Cu at (65.9, 74.6)
Connections:
- U1 pad 24: Net-(U1-Pad24) -> (no net)
- U1 pad 25: Net-(U1-Pad25) -> (no net)
- U1 pad 26: Net-(U1-Pad26) -> (no net)
- U1 pad 27: Net-(U1-Pad27) -> (no net)
- U1 pad 28: Net-(U1-Pad28) -> (no net)
- U1 pad 29: Net-(U1-Pad29) -> (no net)
- U1 pad 3: Net-(U1-Pad3) -> GND
- U1 pad 4: Net-(U1-Pad4) -> GND
Routing:
- net ROW2: track 185.6 -> 204.6 mm
- net Net-(D29-Pad2): track 0.00 -> 9.74 mm
- net Net-(D27-Pad2): track 0.00 -> 9.74 mm
- net COL6: track 206.6 -> 209.6 mm
- net COL8: track 263.9 -> 266.9 mm
