File: PCBs/wren-plain/wren-plain.kicad_pcb (KiCad board)
At the start: 2 copper layers, 149.1 x 112.8 mm, 71 parts, among them J1 TRRS_Jack, SW0 Reset, U1 Elite-C

Commit message: Standardize MCU Pins
Parts:
- removed the G*** at (241.3, 76.4) (x2)
- added G***: LOGO, footprints:wren_logo, B.Cu at (241.3, 76.4)
- added G***: LOGO, footprints:wren_logo, F.Cu at (241.3, 76.4)
Connections:
- U1 pad 10: RIGHT -> LEFT
- U1 pad 11: Net-(U1-Pad11) -> RIGHT
- U1 pad 19: Net-(U1-Pad19) -> (no net)
- U1 pad 20: Net-(U1-Pad20) -> (no net)
- U1 pad 24: Net-(U1-Pad24) -> (no net)
- U1 pad 25: Net-(U1-Pad25) -> (no net)
- U1 pad 26: Net-(U1-Pad26) -> (no net)
- U1 pad 27: Net-(U1-Pad27) -> (no net)
- U1 pad 28: Net-(U1-Pad28) -> (no net)
- U1 pad 29: Net-(U1-Pad29) -> (no net)
- U1 pad 9: LEFT -> (no net)
Routing:
- net Net-(D36-Pad2): track 6.50 -> 9.56 mm
- net RIGHT: track 181.8 -> 182.8 mm
- net LEFT: track 182.2 -> 183.3 mm
