File: PCBs/wren-pcb/wren-pcb.kicad_pcb (KiCad board)
At the start: 2 copper layers, 227.7 x 112.8 mm, 117 parts, among them J1 TRRS_Jack, SW0 Reset, U1 Elite-C

Commit message: Continue working
Parts:
- moved FID14 0.73 mm to (55.2, 42.7)
- moved FID13 0.67 mm to (55.2, 49.2)
- moved FID6 0.67 mm to (114.8, 49.2)
- moved FID10 0.67 mm to (55.2, 87.3)
- moved FID9 0.67 mm to (114.8, 87.3)
- moved FID4 0.60 mm to (114.8, 42.9)
- moved FID11 0.60 mm to (55.2, 81.0)
- moved FID7 0.60 mm to (114.8, 81.0)
Routing:
- net COL2: track 15.3 -> 158.4 mm, vias 0 -> 1
- net COL0: track 32.8 -> 123.5 mm
- net COL1: track 53.7 -> 136.7 mm
- net COL3: track 98.9 -> 180.5 mm
- net COL4: track 12.9 -> 92.5 mm
- net COL6: track 155.4 -> 211.2 mm
- net COL9: track 229.8 -> 284.7 mm
- net COL7: track 23.5 -> 77.7 mm
- net COL5: track 12.3 -> 66.5 mm
- net COL8: track 42.6 -> 96.7 mm
- net ROW3: track 0.24 -> 31.6 mm
- net Net-(D41-Pad2): track 2.91 -> 10.7 mm
- net Net-(D43-Pad2): track 3.07 -> 10.7 mm
- net Net-(D44-Pad2): track 3.07 -> 10.7 mm
- net Net-(D42-Pad2): track 3.07 -> 10.4 mm
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Other:
- outline, holes or cut-outs redrawn
