File: PCBs/wren-universal-2.0/wren-universal.kicad_pcb (KiCad board)
At the start: 2 copper layers, 227.7 x 112.8 mm, 121 parts, among them J1 TRRS_Jack, J2 Nice!Nano Compatibility, SW0 Reset, U1 Elite-C, U2 EGG PRO MICRO

Commit message: Add battery header, update readme
Parts:
- added BT1: Battery_Cell, Connector_PinHeader_2.00mm:PinHeader_1x02_P2.00mm_Vertical, B.Cu at (232.2, 56.7)
Connections:
- U1 pad 23: GND -> BATT-
- U1 pad 24: unconnected-(U1-B0-Pad24) -> BATT+
- U1 pad 3: unconnected-(U1-GND-Pad3) -> GND
Routing:
- net GND: track 222.4 -> 228.0 mm, vias 2 -> 3
- net BATT-: track 0.00 -> 4.73 mm
- net BATT+: track 0.00 -> 3.50 mm
Changed lines of the file:
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@@
   (net 66 "Net-(U1-RST)")
   (net 67 "ENC1-IN")
-  (net 68 "unconnected-(U1-GND-Pad3)")
+  (net 68 "BATT+")
   (net 69 "unconnected-(U1-GND-Pad4)")
-  (net 70 "unconnected-(U1-B0-Pad24)")
+  (net 70 "BATT-")
   (net 71 "unconnected-(U1-B7-Pad25)")
   (net 72 "unconnected-(U1-D5-Pad26)")
@@
         (effects (font (size 1 1) (thickness 0.15)))
     )
+    (fp_text user "${REFERENCE}" (at 0 2.54 180) (layer "F.Fab") hide
+        (effects (font (size 1 1) (thickness 0.15)))
+    )
     (fp_line (start -1.33 -1.33) (end 0 -1.33)
       (stroke (width 0.12) (type solid)) (layer "F.SilkS"))
@@
     (fp_line (start 1.33 1.27) (end 1.33 6.41)
       (stroke (width 0.12) (type solid)) (layer "F.SilkS"))
+    (fp_line (start -1.8 -1.8) (end -1.8 6.85)
+      (stroke (width 0.05) (type solid)) (layer "F.CrtYd"))
+    (fp_line (start -1.8 6.85) (end 1.8 6.85)
+      (stroke (width 0.05) (type solid)) (layer "F.CrtYd"))
+    (fp_line (start 1.8 -1.8) (end -1.8 -1.8)
+      (stroke (width 0.05) (type solid)) (layer "F.CrtYd"))
+    (fp_line (start 1.8 6.85) (end 1.8 -1.8)
+      (stroke (width 0.05) (type solid)) (layer "F.CrtYd"))
     (fp_line (start -1.27 -0.635) (end -0.635 -1.27)
       (stroke (width 0.1) (type solid)) (layer "F.Fab"))
@@
       (net 13 "ROW1") (pinfunction "RX1/PD2") (pintype "input"))
     (pad "3" thru_hole circle (at -8.89 -7.62 270) (size 1.7526 1.7526) (drill 1.0922) (layers "*.Cu" "*.SilkS" "*.Mask")
-      (net 68 "unconnected-(U1-GND-Pad3)") (pinfunction "GND") (pintype "input+no_connect"))
+      (net 62 "GND") (pinfunction "GND") (pintype "input"))
     (pad "4" thru_hole circle (at -6.35 -7.62 270) (size 1.7526 1.7526) (drill 1.0922) (layers "*.Cu" "*.SilkS" "*.Mask")
       (net 69 "unconnected-(U1-GND-Pad4)") (pinfunction "GND") (pintype "input+no_connect"))
@@
       (net 66 "Net-(U1-RST)") (pinfunction "RST") (pintype "input"))
     (pad "23" thru_hole circle (at -11.43 7.62 270) (size 1.7526 1.7526) (drill 1.0922) (layers "*.Cu" "*.SilkS" "*.Mask")
-      (net 62 "GND") (pinfunction "GND") (pintype "input"))
+      (net 70 "BATT-") (pinfunction "GND") (pintype "input"))
     (pad "24" thru_hole circle (at -13.97 7.62 270) (size 1.7526 1.7526) (drill 1.0922) (layers "*.Cu" "*.SilkS" "*.Mask")
-      (net 70 "unconnected-(U1-B0-Pad24)") (pinfunction "B0") (pintype "input+no_connect"))
+      (net 68 "BATT+") (pinfunction "B0") (pintype "input"))
     (pad "25" thru_hole circle (at 13.97 -5.08 270) (size 1.7526 1.7526) (drill 1.0922) (layers "*.Cu" "*.SilkS" "*.Mask")
       (net 71 "unconnected-(U1-B7-Pad25)") (pinfunction "B7") (pintype "input+no_connect"))
@@
       (net 90 "unconnected-(U2-B0-Pad24)") (pinfunction "B0") (pintype "input+no_connect"))
   )
+  (footprint "Connector_PinHeader_2.00mm:PinHeader_1x02_P2.00mm_Vertical" (layer "B.Cu")
+    (at 232.20875 56.7175 180)
+    (descr "Through hole straight pin header, 1x02, 2.00mm pitch, single row")
+    (tags "Through hole pin header THT 1x02 2.00mm single row")
+    (property "Sheetfile" "wren-universal.kicad_sch")
+    (property "Sheetname" "")
+    (property "ki_description" "Single-cell battery")
+    (property "ki_keywords" "battery cell")
+    (attr through_hole)
+    (fp_text reference "BT1" (at 0 2.06) (layer "B.SilkS")
+        (effects (font (size 1 1) (thickness 0.15)) (justify mirror))
+    )
+    (fp_text value "Battery_Cell" (at 0 -4.06) (layer "B.Fab")
+        (effects (font (size 1 1) (thickness 0.15)) (justify mirror))
+    )
+    (fp_text user "${REFERENCE}" (at 0 -1 90) (layer "B.Fab")
+        (effects (font (size 1 1) (thickness 0.15)) (justify mirror))
+    )
+    (fp_line (start -1.06 -3.06) (end 1.06 -3.06)
+      (stroke (width 0.12) (type solid)) (layer "B.SilkS"))
+    (fp_line (start -1.06 -1) (end -1.06 -3.06)
+      (stroke (width 0.12) (type solid)) (layer "B.SilkS"))
+    (fp_line (start -1.06 -1) (end 1.06 -1)
+      (stroke (width 0.12) (type solid)) (layer "B.SilkS"))
+    (fp_line (start -1.06 0) (end -1.06 1.06)
+      (stroke (width 0.12) (type solid)) (layer "B.SilkS"))
+    (fp_line (start -1.06 1.06) (end 0 1.06)
+      (stroke (width 0.12) (type solid)) (layer "B.SilkS"))
+    (fp_line (start 1.06 -1) (end 1.06 -3.06)
+      (stroke (width 0.12) (type solid)) (layer "B.SilkS"))
+    (fp_line (start -1.5 -3.5) (end 1.5 -3.5)
+      (stroke (width 0.05) (type solid)) (layer "B.CrtYd"))
+    (fp_line (start -1.5 1.5) (end -1.5 -3.5)
+      (stroke (width 0.05) (type solid)) (layer "B.CrtYd"))
+    (fp_line (start 1.5 -3.5) (end 1.5 1.5)
+      (stroke (width 0.05) (type solid)) (layer "B.CrtYd"))
+    (fp_line (start 1.5 1.5) (end -1.5 1.5)
+      (stroke (width 0.05) (type solid)) (layer "B.CrtYd"))
+    (fp_line (start -1 -3) (end -1 0.5)
+      (stroke (width 0.1) (type solid)) (layer "B.Fab"))
+    (fp_line (start -1 0.5) (end -0.5 1)
+      (stroke (width 0.1) (type solid)) (layer "B.Fab"))
+    (fp_line (start -0.5 1) (end 1 1)
+      (stroke (width 0.1) (type solid)) (layer "B.Fab"))
+    (fp_line (start 1 -3) (end -1 -3)
+      (stroke (width 0.1) (type solid)) (layer "B.Fab"))
+    (fp_line (start 1 1) (end 1 -3)
+      (stroke (width 0.1) (type solid)) (layer "B.Fab"))
+    (pad "1" thru_hole rect (at 0 0 180) (size 1.35 1.35) (drill 0.8) (layers "*.Cu" "*.Mask")
+      (net 68 "BATT+") (pinfunction "+") (pintype "passive"))
+    (pad "2" thru_hole oval (at 0 -2 180) (size 1.35 1.35) (drill 0.8) (layers "*.Cu" "*.Mask")
+      (net 70 "BATT-") (pinfunction "-") (pintype "passive"))
+    (model "${KICAD6_3DMODEL_DIR}/Connector_PinHeader_2.00mm.3dshapes/PinHeader_1x02_P2.00mm_Vertical.wrl"
+      (offset (xyz 0 0 0))
+      (scale (xyz 1 1 1))
+      (rotate (xyz 0 0 0))
+    )
+  )
   (gr_line (start 232.0835 50.3555) (end 232.0835 51.14925)
     (stroke (width 0.05) (type solid)) (layer "Edge.Cuts"))
@@
   (segment (start 255.631865 117.017615) (end 255.631865 119.462122) (width 0.25) (layer "F.Cu") (net 62))
   (segment (start 246.4665 107.85225) (end 255.631865 117.017615) (width 0.25) (layer "F.Cu") (net 62))
+  (segment (start 241.03525 62.1075) (end 241.07875 62.1075) (width 0.25) (layer "F.Cu") (net 62))
   (segment (start 156.74901 90.25974) (end 156.74901 125.82935) (width 0.25) (layer "F.Cu") (net 62))
-  (segment (start 239.463699 63.679051) (end 235.585 59.800352) (width 0.25) (layer "F.Cu") (net 62))
   (segment (start 159.307 142.874149) (end 159.601824 142.874153) (width 0.25) (layer "F.Cu") (net 62))
+  (segment (start 239.463699 63.679051) (end 241.03525 62.1075) (width 0.25) (layer "F.Cu") (net 62))
   (segment (start 246.4665 93.74925) (end 246.4665 107.85225) (width 0.25) (layer "F.Cu") (net 62))
   (segment (start 159.307 128.38734) (end 159.307 143.30975) (width 0.25) (layer "F.Cu") (net 62))
-  (segment (start 235.585 59.800352) (end 235.585 59.563) (width 0.25) (layer "F.Cu") (net 62))
   (segment (start 239.463699 86.785447) (end 239.463699 63.679051) (width 0.25) (layer "F.Cu") (net 62))
   (segment (start 255.631865 119.462122) (end 255.237717 119.85627) (width 0.25) (layer "F.Cu") (net 62))
@@
   (via (at 239.975501 87.297249) (size 0.8) (drill 0.4) (layers "F.Cu" "B.Cu") (net 62))
   (via (at 157.024 90.019858) (size 0.8) (drill 0.4) (layers "F.Cu" "B.Cu") (net 62))
-  (segment (start 235.585 59.563) (end 235.585 60.325074) (width 0.25) (layer "B.Cu") (net 62))
+  (via (at 241.07875 62.1075) (size 0.8) (drill 0.4) (layers "F.Cu" "B.Cu") (net 62))
   (segment (start 215.497088 88.194298) (end 219.523269 88.194299) (width 0.25) (layer "B.Cu") (net 62))
   (segment (start 239.9605 93.69425) (end 240.0155 93.74925) (width 0.25) (layer "B.Cu") (net 62))
@@
   (segment (start 194.975471 85.451269) (end 212.75406 85.45127) (width 0.25) (layer "B.Cu") (net 62))
   (segment (start 255.237717 119.85627) (end 256.225986 119.85627) (width 0.25) (layer "B.Cu") (net 62))
+  (segment (start 241.07875 62.1075) (end 241.08325 62.103) (width 0.25) (layer "B.Cu") (net 62))
   (segment (start 181.997772 82.0378) (end 191.562 82.0378) (width 0.25) (layer "B.Cu") (net 62))
   (segment (start 239.628432 87.644318) (end 239.975501 87.297249) (width 0.25) (layer "B.Cu") (net 62))
@@
   (segment (start 160.73721 84.49777) (end 174.32762 84.49777) (width 0.25) (layer "B.Cu") (net 62))
   (segment (start 191.562 82.0378) (end 194.975471 85.451269) (width 0.25) (layer "B.Cu") (net 62))
+  (segment (start 241.08325 62.103) (end 250.825 62.103) (width 0.25) (layer "B.Cu") (net 62))
   (segment (start 157.024 90.019858) (end 157.95 89.093858) (width 0.25) (layer "B.Cu") (net 62))
   (segment (start 240.0155 93.74925) (end 246.5155 93.74925) (width 0.25) (layer "B.Cu") (net 62))
@@
   (segment (start 161.807 130.92575) (end 163.247 132.36575) (width 0.25) (layer "B.Cu") (net 67))
   (segment (start 161.807 128.80975) (end 161.807 130.92575) (width 0.25) (layer "B.Cu") (net 67))
+  (segment (start 232.51425 57.023) (end 232.20875 56.7175) (width 0.2) (layer "F.Cu") (net 68))
+  (segment (start 235.585 57.023) (end 232.51425 57.023) (width 0.2) (layer "F.Cu") (net 68))
+  (segment (start 233.05425 59.563) (end 232.20875 58.7175) (width 0.25) (layer "F.Cu") (net 70))
+  (segment (start 235.585 59.563) (end 233.05425 59.563) (width 0.25) (layer "F.Cu") (net 70))
+  (segment (start 235.585 59.800352) (end 235.585 59.563) (width 0.25) (layer "F.Cu") (net 70))
+  (segment (start 235.585 59.563) (end 235.585 60.325074) (width 0.25) (layer "B.Cu") (net 70))
 )
