File: PCBs/wren-mx/wren-mx.kicad_pcb (KiCad board)
At the start: 2 copper layers, 227.7 x 112.8 mm, 122 parts, among them J1 TRRS_Jack, J2 Nice!Nano Compatibility, SW0 Reset, U1 Elite-C, U2 EGG PRO MICRO

Commit message: Add first draft of choc board, move to Seeed Xiao on Egg.
Parts:
- U2: value EGG PRO MICRO -> SeeeduinoXIAO; footprint footprints:ARDUINO_PRO_MICRO -> footprints:Seeeduino XIAO-MOUDLE14P-2.54-21X17.8MM
- moved U2 92.7 mm to (18.3, 39.0), turned to 180 degrees
- moved BT1 11.0 mm to (243.2, 57.3)
Connections:
- U2 pad 1: COL6 -> ROW0
- U2 pad 11: unconnected-(U2-8/PB4-Pad11) -> COL6
- U2 pad 13: ROW3 -> unconnected-(U2-GND-Pad13)
- U2 pad 14: ROW2 -> unconnected-(U2-5V-Pad14)
- U2 pad 15: ROW1 -> unconnected-(U2-5V-Pad15)
- U2 pad 2: COL7 -> COL9
- U2 pad 20: ROW0 -> unconnected-(U2-GND-Pad20)
- U2 pad 3: unconnected-(U2-GND-Pad3) -> COL8
- U2 pad 4: unconnected-(U2-GND-Pad4) -> COL7
- U2 pad 5: unconnected-(U2-2/PD1-Pad5) -> ROW1
- U2 pad 6: unconnected-(U2-3/PD0-Pad6) -> ROW2
- U2 pad 7: COL8 -> ROW3
- U2 pad 8: COL9 -> unconnected-(U2-PB09_A7_D7_RX-Pad8)
Routing:
- net COL0: track 0.00 -> 98.7 mm
- net COL1: track 0.00 -> 96.3 mm
- net COL3: track 0.00 -> 93.7 mm
- net COL4: track 0.00 -> 86.5 mm
- net COL2: track 0.00 -> 78.0 mm
- net VCC: track 0.00 -> 68.2 mm
- net COL6: track 0.00 -> 66.5 mm
- net COL8: track 0.00 -> 66.4 mm
- net COL5: track 0.00 -> 66.4 mm
- net COL9: track 0.00 -> 66.4 mm
- net COL7: track 0.00 -> 66.4 mm
- net GND: track 0.00 -> 40.1 mm
- net ROW0: track 0.00 -> 35.9 mm
- net Net-(U1-RST): track 0.00 -> 35.5 mm
- net SDA: track 0.00 -> 15.4 mm
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Other:
- outline, holes or cut-outs redrawn
