File: PCBs/wren-mx/wren-mx.kicad_sch (KiCad schematic)
At the start: 122 parts, among them J1 TRRS_Jack, J2 Nice!Nano Compatibility, SW0 Reset, U1 Elite-C, U2 EGG PRO MICRO

Commit message: Add first draft of choc board, move to Seeed Xiao on Egg.
Parts:
- removed U2: EGG PRO MICRO, footprints:ARDUINO_PRO_MICRO, symbol wren-universal-cache:wren-numpad-rescue_Elite-C-keebio-wren-left-rescue
- added U2: SeeeduinoXIAO, footprints:Seeeduino XIAO-MOUDLE14P-2.54-21X17.8MM, symbol XIAO:SeeeduinoXIAO
Connections:
- net COL6: now also U2.11 (PA6_A10_D10_MOSI)
- net COL7: now also U2.4 (PA11_A3_D3)
- net COL8: now also U2.3 (PA10_A2_D2)
- net COL9: now also U2.2 (PA4_A1_D1)
- net ROW0: now also U2.1 (PA02_A0_D0)
- net ROW1: now also U2.5 (PA8_A4_D4_SDA)
- net ROW2: now also U2.6 (PA9_A5_D5_SCL)
- net ROW3: now also U2.7 (PB08_A6_D6_TX)
- no-connect marks 28 -> 19
Other:
- moved on the sheet: J2
